File: aniol32kiCad/exp.sch (KiCad schematic (older format))
At the start: 1 part

Commit message: lots of changes
Parts:
- gave numbers to parts that had none: 1
Changed lines of the file:
@@
 $Descr A4 11693 8268
 encoding utf-8
-Sheet 5 5
+Sheet 5 4
 Title ""
 Date ""
@@
 $EndDescr
 $Comp
-L Connector:Conn_01x24_Male J?
+L Connector:Conn_01x24_Male J7
 U 1 1 618B4600
 P 5550 2400
-F 0 "J?" H 5658 3681 50  0000 C CNN
+F 0 "J7" H 5658 3681 50  0000 C CNN
 F 1 "Conn_01x24_Male" H 5658 3590 50  0000 C CNN
 F 2 "" H 5550 2400 50  0001 C CNN
