File: aniol32kiCad/aniol32.sch (KiCad schematic (older format))
At the start: 33 parts, among them J1 RST, J2 PWR, J3 Conn_02x08_Odd_Even, U1 74LS32, U12 74LS74, U2 74LS14, U3 74LS14, U4 74LS32, U5 74LS08, U9 DART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

Commit message: Doc changes
Removed a '32 from A32
Documented the VGA connector
Parts:
- removed C14: 100n, Capacitor_THT:C_Disc_D5.0mm_W2.5mm_P5.00mm, symbol Device:C_Small
- removed U1: 74LS32, Package_DIP:DIP-14_W7.62mm_Socket, symbol 74xx:74LS32
- removed U3: 74LS14, Package_DIP:DIP-14_W7.62mm_Socket, symbol 74xx:74LS14
- added unit 1 of U2
- added U6: 74LS02, symbol 74xx:74LS02
- renumbered J3 to SERIAL1
Connections:
- net +5V: now also SERIAL1.2 (Pin_2), U6.14 (VCC); no longer SERIAL1.15 (Pin_15)
- net CLK: now also U2.2
- net GND: now also SERIAL1.15 (Pin_15), U6.7 (GND); no longer SERIAL1.2 (Pin_2)
- net WAIT: now also U9.10 (~W~/~RDYA)
- net at U9.22 (~DCDB): now also SERIAL1.10 (Pin_10); no longer SERIAL1.1 (Pin_1)
- net at X1.8 (OUT): now also U2.1
- no-connect marks 11 -> 10
Changed lines of the file:
@@
 NoConn ~ 2900 2700
-$Comp
-L 74xx:74LS32 U1
-U 5 1 619D9E00
-P 1650 7050
-F 0 "U1" H 1600 7650 50  0000 L CNN
-F 1 "74LS32" H 1500 7050 50  0000 L CNN
-F 2 "Package_DIP:DIP-14_W7.62mm_Socket" H 1650 7050 50  0001 C CNN
-F 3 "http://www.ti.com/lit/gpn/sn74LS32" H 1650 7050 50  0001 C CNN
-	5    1650 7050
-	1    0    0    -1
-$EndComp
 $Comp
 L Device:CP C1
@@
 Wire Wire Line
 	850  6550 1150 6550
-Connection ~ 1650 6550
-Wire Wire Line
-	1650 6550 2100 6550
 Connection ~ 2100 6550
 Wire Wire Line
 	850  7550 850  7200
-Connection ~ 1650 7550
-Wire Wire Line
-	1650 7550 1150 7550
 Connection ~ 2100 7550
-Wire Wire Line
-	2100 7550 1650 7550
 Wire Wire Line
 	850  6550 850  6900
@@
 	1    0    0    -1
 $EndComp
-$Comp
-L 74xx:74LS14 U3
-U 7 1 61D2B7EA
-P 2550 7050
-F 0 "U3" H 2450 7650 50  0000 L CNN
-F 1 "74LS14" H 2450 7050 50  0000 L CNN
-F 2 "Package_DIP:DIP-14_W7.62mm_Socket" H 2550 7050 50  0001 C CNN
-F 3 "http://www.ti.com/lit/gpn/sn74LS14" H 2550 7050 50  0001 C CNN
-	7    2550 7050
-	1    0    0    -1
-$EndComp
-Connection ~ 2550 6550
-Wire Wire Line
-	2550 6550 3000 6550
-Connection ~ 2550 7550
-Wire Wire Line
-	2550 7550 3000 7550
 Connection ~ 3450 7550
 Connection ~ 3000 6550
 Connection ~ 3000 7550
-Wire Wire Line
-	2100 6550 2550 6550
-Wire Wire Line
-	2100 7550 2550 7550
 Wire Wire Line
 	3000 7550 3450 7550
@@
 $EndComp
 $Comp
-L 74xx:74LS14 U3
-U 3 1 61D3D610
-P 3800 5100
-F 0 "U3" H 3800 5417 50  0000 C CNN
-F 1 "74LS14" H 3800 5326 50  0000 C CNN
-F 2 "Package_DIP:DIP-14_W7.62mm_Socket" H 3800 5100 50  0001 C CNN
-F 3 "http://www.ti.com/lit/gpn/sn74LS14" H 3800 5100 50  0001 C CNN
-	3    3800 5100
-	1    0    0    -1
-$EndComp
-$Comp
 L power:+5V #PWR014
 U 1 1 61D3E347
@@
 	1    0    0    -1
 $EndComp
-$Comp
-L Device:C_Small C14
-U 1 1 61D458CD
-P 6100 7100
-F 0 "C14" H 6050 7300 50  0000 L CNN
-F 1 "100n" H 6000 6950 50  0000 L CNN
-F 2 "Capacitor_THT:C_Disc_D5.0mm_W2.5mm_P5.00mm" H 6100 7100 50  0001 C CNN
-F 3 "~" H 6100 7100 50  0001 C CNN
-	1    6100 7100
-	1    0    0    -1
-$EndComp
 Wire Wire Line
 	3900 7550 4300 7550
@@
 Wire Wire Line
 	5800 7000 5950 7000
-Connection ~ 5950 7000
-Wire Wire Line
-	5950 7000 6100 7000
 Wire Wire Line
 	4300 7200 4450 7200
@@
 Wire Wire Line
 	5800 7200 5950 7200
-Connection ~ 5950 7200
-Wire Wire Line
-	5950 7200 6100 7200
 $Comp
 L Connector:Conn_01x02_Male J2
@@
 L power:GND #PWR0103
 U 1 1 61DB4965
-P 10950 2650
-F 0 "#PWR0103" H 10950 2400 50  0001 C CNN
-F 1 "GND" H 10955 2477 50  0000 C CNN
-F 2 "" H 10950 2650 50  0001 C CNN
-F 3 "" H 10950 2650 50  0001 C CNN
-	1    10950 2650
+P 10100 1250
+F 0 "#PWR0103" H 10100 1000 50  0001 C CNN
+F 1 "GND" H 10105 1077 50  0000 C CNN
+F 2 "" H 10100 1250 50  0001 C CNN
+F 3 "" H 10100 1250 50  0001 C CNN
+	1    10100 1250
 	1    0    0    -1
 $EndComp
@@
 L power:+5V #PWR0104
 U 1 1 61DB55FD
-P 10250 1450
-F 0 "#PWR0104" H 10250 1300 50  0001 C CNN
-F 1 "+5V" H 10265 1623 50  0000 C CNN
-F 2 "" H 10250 1450 50  0001 C CNN
-F 3 "" H 10250 1450 50  0001 C CNN
-	1    10250 1450
+P 11050 1350
+F 0 "#PWR0104" H 11050 1200 50  0001 C CNN
+F 1 "+5V" H 11065 1523 50  0000 C CNN
+F 2 "" H 11050 1350 50  0001 C CNN
+F 3 "" H 11050 1350 50  0001 C CNN
+	1    11050 1350
 	1    0    0    -1
 $EndComp
@@
 NoConn ~ 9650 2500
 Wire Wire Line
-	9650 2850 10350 2850
-Wire Wire Line
 	9650 2650 10250 2650
 Wire Wire Line
@@
 	9650 3450 10850 3450
 Wire Wire Line
-	11150 3550 11150 2000
-Wire Wire Line
-	11150 2000 10950 2000
-Wire Wire Line
-	9650 3550 11150 3550
-Wire Wire Line
 	9650 1550 10850 1550
 Wire Wire Line
@@
 	10850 3450 10850 2650
 Wire Wire Line
-	10250 1450 10250 2150
-Wire Wire Line
-	10950 2150 10950 2000
-Wire Wire Line
 	10850 1550 10850 2150
 Wire Wire Line
@@
 	10350 2150 10350 2100
 Wire Wire Line
-	10350 2100 9850 2100
-Wire Wire Line
-	9850 2100 9850 2750
-Wire Wire Line
-	9850 2750 10000 2750
-Wire Wire Line
-	9650 2750 9850 2750
-Connection ~ 9850 2750
+	10350 2100 9950 2100
+Wire Wire Line
+	9950 2100 9950 2750
 Wire Wire Line
 	7900 4500 7900 4900
@@
 $EndComp
 Connection ~ 1150 6550
-Wire Wire Line
-	1150 6550 1650 6550
 $Comp
 L power:PWR_FLAG #FLG0102
@@
 Wire Wire Line
 	2550 2800 2450 2800
-Text GLabel 9650 3050 2    50   Input ~ 0
+Text GLabel 10200 3050 2    50   Input ~ 0
 WAIT
-NoConn ~ 10550 2650
-NoConn ~ 9650 2050
 Text GLabel 6100 3350 0    50   Input ~ 0
 MEMRQ
 NoConn ~ 4300 3100
-$Comp
-L Connector_Generic:Conn_02x08_Odd_Even J3
+Wire Wire Line
+	9650 3550 10550 3550
+Wire Wire Line
+	10200 3050 9750 3050
+Wire Wire Line
+	9650 2050 9750 2050
+$Comp
+L Connector_Generic:Conn_02x08_Odd_Even SERIAL1
 U 1 1 621728BB
 P 10650 2350
-F 0 "J3" V 10654 2730 50  0000 L CNN
-F 1 "Conn_02x08_Odd_Even" V 10745 2730 50  0000 L CNN
+F 0 "SERIAL1" H 10600 1850 50  0000 L CNN
+F 1 "Conn_02x08_Odd_Even" V 10700 1850 50  0000 L CNN
 F 2 "Connector_PinSocket_2.54mm:PinSocket_2x08_P2.54mm_Horizontal" H 10650 2350 50  0001 C CNN
 F 3 "~" H 10650 2350 50  0001 C CNN
@@
 	0    1    1    0
 $EndComp
+Wire Wire Line
+	10550 2650 10550 3550
+Connection ~ 9950 2750
+Wire Wire Line
+	9950 2750 10000 2750
+Wire Wire Line
+	9650 2750 9950 2750
+NoConn ~ 10950 2150
+Wire Wire Line
+	9650 2850 10350 2850
+Wire Wire Line
+	9750 2050 9750 3050
+Connection ~ 9750 3050
+Wire Wire Line
+	9750 3050 9650 3050
+Wire Wire Line
+	10100 1250 10250 1250
+Wire Wire Line
+	10250 1250 10250 2150
+Wire Wire Line
+	10950 2650 11050 2650
+Wire Wire Line
+	11050 2650 11050 1350
+$Comp
+L 74xx:74LS14 U2
+U 1 1 621EE5D7
+P 3800 5100
+F 0 "U2" H 3800 5417 50  0000 C CNN
+F 1 "74LS14" H 3800 5326 50  0000 C CNN
+F 2 "Package_DIP:DIP-14_W7.62mm_Socket" H 3800 5100 50  0001 C CNN
+F 3 "http://www.ti.com/lit/gpn/sn74LS14" H 3800 5100 50  0001 C CNN
+	1    3800 5100
+	1    0    0    -1
+$EndComp
+Wire Wire Line
+	2100 6550 2550 6550
+Wire Wire Line
+	2100 7550 2550 7550
+Wire Wire Line
+	1150 6550 2100 6550
+Wire Wire Line
+	1150 7550 2100 7550
+$Comp
+L 74xx:74LS02 U6
+U 5 1 62234E1C
+P 2550 7050
+F 0 "U6" H 2450 7650 50  0000 L CNN
+F 1 "74LS02" H 2450 7050 50  0000 L CNN
+F 2 "" H 2550 7050 50  0001 C CNN
+F 3 "http://www.ti.com/lit/gpn/sn74ls02" H 2550 7050 50  0001 C CNN
+	5    2550 7050
+	1    0    0    -1
+$EndComp
+Connection ~ 2550 6550
+Wire Wire Line
+	2550 6550 3000 6550
+Connection ~ 2550 7550
+Wire Wire Line
+	2550 7550 3000 7550
 $EndSCHEMATC
