File: aniol32kiCad/aniol32.sch (KiCad schematic (older format))
At the start: 31 parts, among them J1 RST, J2 PWR, U12 74LS74, U2 74LS14, U4 74LS32, U5 74LS08, U6 74LS02, U9 DART, X1 ACO-1.8432MHz

Commit message: developing the skbd module
Parts:
- removed C10, C11, C12, C13, C9: 100n, Capacitor_THT:C_Disc_D5.0mm_W2.5mm_P5.00mm, symbol Device:C_Small
- removed R1: 4k7, Resistor_THT:R_Axial_DIN0207_L6.3mm_D2.5mm_P7.62mm_Horizontal, symbol Device:R_Small
- removed SERIAL1: Conn_02x08_Odd_Even, Connector_PinSocket_2.54mm:PinSocket_2x08_P2.54mm_Horizontal, symbol Connector_Generic:Conn_02x08_Odd_Even
- removed U5: 74LS08, Package_DIP:DIP-14_W7.62mm_Socket, symbol 74xx:74LS08
- removed U6: 74LS02, symbol 74xx:74LS02
- removed U9: DART, Package_DIP:DIP-40_W15.24mm_Socket, symbol Zilog_Z80_Peripherals:DART-DIP-40
- added R?: 4k7, Resistor_THT:R_Axial_DIN0207_L6.3mm_D2.5mm_P7.62mm_Horizontal, symbol Device:R
- added RAM: 6116, symbol memory:6116
- added U?: 74LS32, symbol 74xx:74LS32
- added U?: 74LS14, symbol 74xx:74LS14
Connections:
- net +5V: now also ROM1.27 (~WE), R?.2, RAM.24 (VCC)
- net A0: now also RAM.8 (A0)
- net A1: now also RAM.7 (A1)
- net A10: now also RAM.19 (A10)
- net A2: now also RAM.6 (A2)
- net A3: now also RAM.5 (A3)
- net A4: now also RAM.4 (A4)
- net A5: now also RAM.3 (A5)
- net A6: now also RAM.2 (A6)
- net A7: now also RAM.1 (A7)
- net A8: now also RAM.23 (A8)
- net A9: now also RAM.22 (A9)
- net D0: now also RAM.9 (Q0)
- net D1: now also RAM.10 (Q1)
- net D2: now also RAM.11 (Q2)
- net D3: now also RAM.13 (Q3)
- net D4: now also RAM.14 (Q4)
- net D5: now also RAM.15 (Q5)
- net D6: now also RAM.16 (Q6)
- net D7: now also RAM.17 (Q7)
- net GND: now also RAM.12 (GND)
- net INT: now also R?.1
- net MEMRQ: now also ROM1.22 (~OE), U?.12; no longer ROM1.20 (~CS)
- net RD: now also RAM.20 (~OE); no longer ROM1.22 (~OE)
- net WR: now also RAM.21 (~WE); no longer ROM1.27 (~WE)
- net A15: now reaches CPU1.5 (A15)
- net A15: now also ROM1.20 (~CS), U?.1
- new net: RAM.18 (~CS), U?.11
- new net: U?.13, U?.2
- no-connect marks 9 -> 4
Other:
- moved on the sheet: EXP_PORT1, J1, J2, R2, U2A, X1
