File: aniol32kiCad/file6262EA80.sch (KiCad schematic (older format))
At the start: 3 parts

Commit message: moved dev drivers and utils to separate folders
Parts:
- gave numbers to parts that had none: 1
Changed lines of the file:
@@
 	2850 2100 2950 2100
 $Comp
-L Connector_Generic:Conn_02x08_Odd_Even SERIAL?
+L Connector_Generic:Conn_02x08_Odd_Even SERIAL
 U 1 1 62639475
 P 3850 2400
-F 0 "SERIAL?" H 3800 1900 50  0000 L CNN
+F 0 "SERIAL" H 3750 1850 50  0000 L CNN
 F 1 "Conn_02x08_Odd_Even" V 3900 1900 50  0000 L CNN
 F 2 "Connector_PinSocket_2.54mm:PinSocket_2x08_P2.54mm_Horizontal" H 3850 2400 50  0001 C CNN

Commit message: Compact Flash interface
Connections:
- net IO_IEO: now reaches R?.1, U?.6 (IEI)
Changed lines of the file:
@@
 Wire Wire Line
 	4250 2700 4250 1400
+Text GLabel 1650 4350 2    50   Input ~ 0
+IO_IEO
 $EndSCHEMATC
