File: casette/cassetteInterface/z180/z180.sch (KiCad schematic (older format))
At the start: 13 parts, among them IC1 Z8-L180-S180-180-PLCC-68, J1 Barrel_Jack, J2 Conn_Coaxial, J3 Mini-DIN-6, J4 Mini-DIN-6, J5 Conn_02x20_Odd_Even, J6 Conn_01x24_Male, U1 GAL16V8, U2 ATmega8A-PU, U3 AS6C4008-55PCN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

Commit message: Added AniolZ180 CUPL project
Parts:
- removed J3, J4: Mini-DIN-6, symbol Connector:Mini-DIN-6
- added J3: Conn_01x04_Female, Connector_PinHeader_2.54mm:PinHeader_1x04_P2.54mm_Horizontal, symbol Connector:Conn_01x04_Female
- added SW1: SW_Push_SPDT, Button_Switch_THT:SW_Tactile_SKHH_Angled, symbol Switch:SW_Push_SPDT
Connections:
- net A0: now reaches IC1.14 (A0)
- net A0: now also U3.12 (A0), U4.12 (A0)
- net A1: now reaches IC1.15 (A1)
- net A1: now also U3.11 (A1), U4.11 (A1)
- net A2: now reaches IC1.16 (A2)
- net A2: now also U3.10 (A2), U4.10 (A2)
- net A3: now reaches IC1.17 (A3)
- net A3: now also U3.9 (A3), U4.9 (A3)
- net A4: now reaches IC1.19 (A4)
- net A4: now also U3.8 (A4), U4.8 (A4)
- net A5: now reaches IC1.20 (A5)
- net A5: now also U3.7 (A5), U4.7 (A5)
- net A6: now reaches IC1.21 (A6)
- net A6: now also U3.6 (A6), U4.6 (A6)
- net A7: now reaches IC1.22 (A7)
- net A7: now also U3.5 (A7), U4.5 (A7)
- net A8: now reaches IC1.23 (A8)
- net A8: now also U3.27 (A8), U4.27 (A8)
- net A9: now reaches IC1.24 (A9)
- net A9: now also U3.26 (A9), U4.26 (A9)
- net A10: now reaches IC1.25 (A10)
- net A10: now also U3.23 (A10), U4.23 (A10)
- net A11: now reaches IC1.26 (A11)
- net A11: now also U3.25 (A11), U4.25 (A11)
- net A12: now reaches IC1.27 (A12)
- net A12: now also U3.4 (A12), U4.4 (A12)
- net A13: now reaches IC1.28 (A13)
- net A13: now also U3.28 (A13), U4.28 (A13)
- net A14: now reaches IC1.29 (A14)
- net A14: now also U3.3 (A14), U4.29 (A14)
- net A15: now reaches IC1.30 (A15)
- net A15: now also U3.31 (A15), U4.3 (A15)
- net A16: now reaches IC1.31 (A16)
- net A16: now also U3.2 (A16), U4.2 (A16)
- net A17: now reaches IC1.32 (A17)
- net A17: now also U3.30 (A17)
- net A18: now reaches IC1.33 (A18/TOUT)
- net A18: now also U3.1 (A18)
- net A19: now reaches IC1.35 (A19)
- net D0: now reaches IC1.37 (D0)
- net D0: now also IC1.39 (D2), J6.19 (Pin_19), J6.21 (Pin_21), U3.13 (DQ0), U3.15 (DQ2), U4.13 (D0), U4.15 (D2)
- net D1: now reaches IC1.38 (D1)
- net D1: now also J6.20 (Pin_20), U3.14 (DQ1), U4.14 (D1)
- net D3: now reaches IC1.40 (D3)
- net D3: now also J6.18 (Pin_18), U3.17 (DQ3), U4.17 (D3)
- net D4: now reaches IC1.41 (D4)
- net D4: now also J6.17 (Pin_17), U3.18 (DQ4), U4.18 (D4)
- net D5: now reaches IC1.42 (D5)
- net D5: now also J6.16 (Pin_16), U3.19 (DQ5), U4.19 (D5)
- net D6: now reaches IC1.43 (D6)
- net D6: now also J6.15 (Pin_15), U3.20 (DQ6), U4.20 (D6)
- net D7: now reaches IC1.44 (D7)
- net D7: now also J6.14 (Pin_14), U3.21 (DQ7), U4.21 (D7)
Other:
- moved on the sheet: IC1, U3, U4
