File: aniol64kiCad/peri.kicad_sch (KiCad schematic)
At the start: 3 parts

Commit message: added scrolling in edit
Parts:
- R?: value (none) -> 4k7; footprint (none) -> Resistor_THT:R_Axial_DIN0207_L6.3mm_D2.5mm_P7.62mm_Horizontal
- SERIAL?: value (none) -> Conn_02x08_Odd_Even; footprint (none) -> Connector_PinSocket_2.54mm:PinSocket_2x08_P2.54mm_Horizontal
- U?: value (none) -> DART; footprint (none) -> Package_DIP:DIP-40_W15.24mm_Socket
Changed lines of the file:
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@@
     (in_bom yes) (on_board yes)
     (property "Reference" "U?" (id 0) (at 76.2 33.02 0))
-    (property "Value" "" (id 1) (at 66.04 33.02 0))
-    (property "Footprint" "" (id 2) (at 73.66 -12.7 0)
+    (property "Value" "DART" (id 1) (at 66.04 33.02 0))
+    (property "Footprint" "Package_DIP:DIP-40_W15.24mm_Socket" (id 2) (at 73.66 -12.7 0)
       (effects (font (size 1.27 1.27)) (justify left) hide)
     )
@@
       (effects (font (size 1.27 1.27)) hide)
     )
-    (property "Value" "" (id 1) (at 71.247 97.1042 0))
+    (property "Value" "GND" (id 1) (at 71.247 97.1042 0))
     (property "Footprint" "" (id 2) (at 71.12 92.71 0)
       (effects (font (size 1.27 1.27)) hide)
@@
       (effects (font (size 1.27 1.27)) hide)
     )
-    (property "Value" "" (id 1) (at 71.501 24.8158 0))
+    (property "Value" "+5V" (id 1) (at 71.501 24.8158 0))
     (property "Footprint" "" (id 2) (at 71.12 29.21 0)
       (effects (font (size 1.27 1.27)) hide)
@@
       (effects (font (size 1.27 1.27)) (justify left))
     )
-    (property "Value" "" (id 1) (at 46.99 80.01 90)
+    (property "Value" "4k7" (id 1) (at 46.99 80.01 90)
       (effects (font (size 1.27 1.27)) (justify left))
     )
-    (property "Footprint" "" (id 2) (at 49.53 77.47 0)
+    (property "Footprint" "Resistor_THT:R_Axial_DIN0207_L6.3mm_D2.5mm_P7.62mm_Horizontal" (id 2) (at 49.53 77.47 0)
       (effects (font (size 1.27 1.27)) hide)
     )
@@
       (effects (font (size 1.27 1.27)) hide)
     )
-    (property "Value" "" (id 1) (at 95.377 32.3342 0))
+    (property "Value" "GND" (id 1) (at 95.377 32.3342 0))
     (property "Footprint" "" (id 2) (at 95.25 27.94 0)
       (effects (font (size 1.27 1.27)) hide)
@@
       (effects (font (size 1.27 1.27)) hide)
     )
-    (property "Value" "" (id 1) (at 119.761 26.0858 0))
+    (property "Value" "+5V" (id 1) (at 119.761 26.0858 0))
     (property "Footprint" "" (id 2) (at 119.38 30.48 0)
       (effects (font (size 1.27 1.27)) hide)
@@
       (effects (font (size 1.27 1.27)) (justify left))
     )
-    (property "Value" "" (id 1) (at 96.52 57.15 90)
+    (property "Value" "Conn_02x08_Odd_Even" (id 1) (at 96.52 57.15 90)
       (effects (font (size 1.27 1.27)) (justify left))
     )
-    (property "Footprint" "" (id 2) (at 109.22 55.88 0)
+    (property "Footprint" "Connector_PinSocket_2.54mm:PinSocket_2x08_P2.54mm_Horizontal" (id 2) (at 109.22 55.88 0)
       (effects (font (size 1.27 1.27)) hide)
     )
