File: aniol640kiCad/BitmappedGraphicsCard/BitmappedGraphicsCard.kicad_sch (KiCad schematic)
At the start: 29 parts

Commit message: schematic updates
Parts:
- added U? (x2): 74LS574, symbol 74xx:74LS574
- added U?: 74LS74, symbol 74xx:74LS74
- added X?: CXO_DIP8, Oscillator:Oscillator_DIP-8, symbol Oscillator:CXO_DIP8
Connections:
- net BgD1 is gone; now on net ClMD4: ColorRam.16 (Q4)
- net BgD2 is gone; now on net ClMD5: ColorRam.17 (Q5)
- net FgD1 is gone; now on net ClMD1: ColorRam.12 (Q1)
- net FgD2 is gone; now on net ClMD2: ColorRam.13 (Q2)
- net ClMD0: now also ColorRam.11 (Q0)
- net ClMD3: now also ColorRam.15 (Q3)
- net ClMD6: now also ColorRam.18 (Q6)
- net LnA0: now also U?.12 (Y6); no longer U?.17 (Y1)
- net LnA1: now also U?.11 (Y7); no longer U?.16 (Y2)
- net LnA2: now also U?.18 (Y0); no longer U?.15 (Y3)
- net LnA3: now also U?.17 (Y1); no longer U?.14 (Y4)
- net LnA4: now also U?.16 (Y2)
- net LnA5: now also U?.15 (Y3)
- net LnA6: now also U?.14 (Y4)
- net PxClock: now also HCounter.10 (CLK), U?.11 (Cp), U?.5 (Q); no longer HCounter.9 (Q0)
- net VMA6: now also U?.9 (S1); no longer U?.12 (Y6)
- net VMA7: now also U?.6 (S2); no longer U?.11 (Y7)
- net VMA8: now also U?.2 (S3); no longer U?.18 (Y0)
- net at U?.11 (D0): now also U?.2 (D0)
- net at U?.12 (D1): now also U?.3 (D1)
- net at U?.13 (D2): now also U?.4 (D2)
- net at U?.15 (D3): now also U?.5 (D3)
- net at U?.16 (D4): now also U?.6 (D4)
- net at HCounter.4 (Q6), U?.7 (A3): now also R?.2; no longer R?.2
- net INTENSITY: now reaches U?.12 (Zd)
- net at U?.13 (I1d): now also U?.12 (Q7)
- net at U?.14 (I0d): now also U?.13 (Q6)
- net at HCounter.5 (Q3): now also R?.2, U?.10 (A0)
- removed net BgD0: ColorRam.15 (Q3), U?.10 (I1c), U?.3 (I1a), U?.6 (I1b)
- removed net FgD0: ColorRam.11 (Q0), U?.11 (I0c), U?.2 (I0a), U?.5 (I0b)
- new net: HCounter.12 (Q8), R?.2, U?.5 (A5)
- new net: HCounter.13 (Q7), R?.2, U?.6 (A4)
- new net: HCounter.2 (Q5), R?.2, U?.8 (A2)
- new net: HCounter.3 (Q4), R?.2, U?.9 (A1)
- new net: U?.1 (OE), U?.10 (GND)
- new net: U?.3 (C), X?.5 (OUT)
- new net: U?.10 (I1c), U?.14 (Q5)
- new net: U?.11 (I0c), U?.15 (Q4)
- new net: U?.19 (Q0), U?.2 (I0a)
- new net: U?.18 (Q1), U?.3 (I1a)
- new net: U?.17 (Q2), U?.5 (I0b)
- new net: U?.16 (Q3), U?.6 (I1b)
- new net: U?.2 (D), U?.6 (~{Q})
- now unconnected: HCounter.14 (Q9)
- no-connect marks 10 -> 17
Other:
- moved on the sheet: ColorRam, HCounter, PixelRam, R?, U?, VCounter
