File: aniol640kiCad/BitmappedGraphicsCard/8085/8085.kicad_sch (KiCad schematic)
At the start: 3 parts

Commit message: schematic updates
Parts:
- removed U?: 27C256, Package_DIP:DIP-28_W15.24mm, symbol Memory_EPROM:27C256
- added U? (x3): 74LS14, symbol 74xx:74LS14
- added U?: 74HCT541, symbol 74xx:74HCT541
- added U?: 2732, symbol memory:2732
- added U? (x4): 74LS08, symbol 74xx:74LS08
Connections:
- net GND: now also U?.12 (GND)
- net at U?.28 (A15): now also U?.20 (~{G})
- net at U?.34 (IO/~{M}): now also U?.18 (~{E}), U?.3
- net at U?.12 (AD0): now also U?.2 (D0)
- net at U?.13 (AD1): now also U?.3 (D1)
- net at U?.14 (AD2): now also U?.4 (D2)
- net at U?.15 (AD3): now also U?.5 (D3)
- net WR: now reaches U?.31 (~{WR})
- net WR: now also U?.13
- net RD: now reaches U?.32 (~{RD})
- net RD: now also U?.12, U?.19 (G2)
- new net: U?.1, U?.6
- new net: U?.1 (G1), U?.2
- new net: U?.11, U?.5
- new net: U?.13, U?.6
- new net: U?.12, U?.8
- new net A8: U?.10
- new net A9: U?.4
- new net IO/M: U?.5, U?.9
- new net LCD: U?.11
- new net Vcc: U?.24 (Vcc)
