File: A32kiCad/aniol32.sch (KiCad schematic (older format))
At the start: 25 parts, among them J1 RST, J2 PWR, U12 74LS74, U2 74LS14, U4 74LS32, X1 ACO-1.8432MHz

Commit message: Refactored NMI handler
Also, fixed the greeting reverse colour bug
Parts:
- removed C1: 100u, Capacitor_THT:CP_Radial_D14.0mm_P7.50mm, symbol Device:CP
- removed C2, C3, C4, C5, C6, C7, C8: 100n, Capacitor_THT:C_Disc_D5.0mm_W2.5mm_P5.00mm, symbol Device:C_Small
- removed CPU1: Z80, Package_DIP:DIP-40_W15.24mm_Socket, symbol CPU:Z80CPU
- removed EXP_PORT1: Conn_01x24_Male, Connector_PinHeader_2.54mm:PinHeader_1x24_P2.54mm_Horizontal, symbol Connector:Conn_01x24_Male
- removed J1: RST, Connector_PinHeader_2.54mm:PinHeader_1x02_P2.54mm_Vertical, symbol Connector:Conn_01x02_Male
- removed J2: PWR, Connector_PinHeader_2.54mm:PinHeader_1x02_P2.54mm_Vertical, symbol Connector:Conn_01x02_Male
- removed R11, R13, R?: 4k7, Resistor_THT:R_Axial_DIN0207_L6.3mm_D2.5mm_P7.62mm_Horizontal, symbol Device:R
- removed R14: 1k, Resistor_THT:R_Axial_DIN0207_L6.3mm_D2.5mm_P7.62mm_Horizontal, symbol Device:R
- removed R2: 4k7, Resistor_THT:R_Axial_DIN0207_L6.3mm_D2.5mm_P7.62mm_Horizontal, symbol Device:R_Small
- removed RAM: 6116, symbol memory:6116
- removed ROM1: 28C256, Package_DIP:DIP-28_W15.24mm_Socket, symbol Memory_EEPROM:28C256
- removed U12: 74LS74, Package_DIP:DIP-14_W7.62mm_Socket, symbol 74xx:74LS74
- removed U2: 74LS14, Package_DIP:DIP-14_W7.62mm_Socket, symbol 74xx:74LS14
- removed U4: 74LS32, Package_DIP:DIP-14_W7.62mm_Socket, symbol 74xx:74LS32
- removed U?: 74LS32, symbol 74xx:74LS32
- removed U?: 74LS14, symbol 74xx:74LS14
- removed X1: ACO-1.8432MHz, Oscillator:Oscillator_DIP-14, symbol Oscillator:ACO-xxxMHz
